File: kicad/logic_converter.kicad_sch (KiCad schematic)
At the start: 6 parts, among them U2 6N138

Commit message: split
Parts:
- removed U2: 6N138, symbol Isolator:6N138
- added U3: 6N137, Package_DIP:DIP-8_W7.62mm, symbol Isolator:6N137
Connections:
- net GND: now also U3.5 (GND)
- net RAIL_2: now also U3.3 (C)
- net at C1.1, D2.1 (K), R5.2: now also U3.2 (A)
- net at R6.1: now also U3.7 (EN)
- net 5V: now reaches R6.2, R7.2
- net 5V: now also U3.8 (VCC)
- net DCC: now reaches R7.1
- net DCC: now also U3.6 (VO)
Other:
- note removed: "does not work"
Changed lines of the file:
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@@
+	)
+	(junction
+		(at 151.13 77.47)
+		(diameter 0)
+		(color 0 0 0 0)
 	)
 	(junction
@@
 		(color 0 0 0 0)
 	)
-	(junction
-		(at 151.13 77.47)
-		(diameter 0)
-		(color 0 0 0 0)
-	)
 	(wire
 		(pts
@@
 	(wire
 		(pts
-			(xy 143.51 85.09) (xy 143.51 88.9)
+			(xy 143.51 82.55) (xy 143.51 88.9)
 		)
 		(stroke
@@
 	(wire
 		(pts
-			(xy 160.02 88.9) (xy 168.91 88.9)
+			(xy 160.02 88.9) (xy 177.8 88.9)
 		)
 		(stroke
@@
 	(wire
 		(pts
-			(xy 140.97 77.47) (xy 151.13 77.47)
+			(xy 133.35 92.71) (xy 133.35 95.25)
 		)
 		(stroke
@@
 	(wire
 		(pts
-			(xy 140.97 85.09) (xy 143.51 85.09)
+			(xy 140.97 82.55) (xy 143.51 82.55)
 		)
 		(stroke
@@
 	(wire
 		(pts
-			(xy 140.97 87.63) (xy 140.97 90.17)
-		)
-		(stroke
-			(width 0)
-			(type default)
-		)
-	)
-	(wire
-		(pts
 			(xy 125.73 85.09) (xy 121.92 85.09)
 		)
@@
 	(wire
 		(pts
+			(xy 151.13 67.31) (xy 133.35 67.31)
+		)
+		(stroke
+			(width 0)
+			(type default)
+		)
+	)
+	(wire
+		(pts
 			(xy 111.76 90.17) (xy 111.76 88.9)
 		)
@@
 	(wire
 		(pts
+			(xy 151.13 77.47) (xy 151.13 67.31)
+		)
+		(stroke
+			(width 0)
+			(type default)
+		)
+	)
+	(wire
+		(pts
+			(xy 133.35 67.31) (xy 133.35 72.39)
+		)
+		(stroke
+			(width 0)
+			(type default)
+		)
+	)
+	(wire
+		(pts
 			(xy 151.13 77.47) (xy 151.13 78.74)
 		)
@@
 			(width 0)
 			(type default)
-		)
-	)
-	(text "does not work\n"
-		(exclude_from_sim no)
-		(at 110.744 62.484 0)
-		(effects
-			(font
-				(size 1.27 1.27)
-			)
 		)
 	)
@@
 		)
 	)
+	(hierarchical_label "5V"
+		(shape input)
+		(at 177.8 77.47 0)
+		(fields_autoplaced yes)
+		(effects
+			(font
+				(size 1.27 1.27)
+			)
+			(justify left)
+		)
+	)
 	(hierarchical_label "RAIL_2"
 		(shape input)
@@
 			)
 			(justify right)
+		)
+	)
+	(hierarchical_label "DCC"
+		(shape output)
+		(at 177.8 88.9 0)
+		(fields_autoplaced yes)
+		(effects
+			(font
+				(size 1.27 1.27)
+			)
+			(justify left)
+		)
+	)
+	(symbol
+		(lib_id "Isolator:6N137")
+		(at 133.35 82.55 0)
+		(unit 1)
+		(exclude_from_sim no)
+		(in_bom yes)
+		(on_board yes)
+		(dnp no)
+		(fields_autoplaced yes)
+		(property "Reference" "U3"
+			(at 136.7839 69.85 0)
+			(effects
+				(font
+					(size 1.27 1.27)
+				)
+				(justify left)
+			)
+		)
+		(property "Value" "6N137"
+			(at 136.7839 72.39 0)
+			(effects
+				(font
+					(size 1.27 1.27)
+				)
+				(justify left)
+			)
+		)
+		(property "Footprint" "Package_DIP:DIP-8_W7.62mm"
+			(at 133.35 95.25 0)
+			(effects
+				(font
+					(size 1.27 1.27)
+				)
+				(hide yes)
+			)
+		)
+		(property "Datasheet" "https://docs.broadcom.com/docs/AV02-0940EN"
+			(at 111.76 68.58 0)
+			(effects
+				(font
+					(size 1.27 1.27)
+				)
+				(hide yes)
+			)
+		)
+		(property "Description" "Single High Speed LSTTL/TTL Compatible Optocoupler with enable, dV/dt 1000/us, VCM 10, max 7V VCC, DIP-8"
+			(at 133.35 82.55 0)
+			(effects
+				(font
+					(size 1.27 1.27)
+				)
+				(hide yes)
+			)
+		)
+		(pin "3"
+		)
+		(pin "4"
+		)
+		(pin "5"
+		)
+		(pin "6"
+		)
+		(pin "7"
+		)
+		(pin "8"
+		)
+		(pin "2"
+		)
+		(pin "1"
+		)
+		(instances
+			(project ""
+				(path "/11b6b3e0-6260-4ffa-b9c7-47f3b03473c9/e71ecf15-c300-4c9d-862f-92665ebf3933/d2fa69c2-c3e0-43db-84db-bb1b3a6e2002"
+					(reference "U3")
+					(unit 1)
+				)
+			)
 		)
 	)
@@
 	)
 	(symbol
-		(lib_id "Isolator:6N138")
-		(at 133.35 82.55 0)
-		(unit 1)
-		(exclude_from_sim no)
-		(in_bom yes)
-		(on_board yes)
-		(dnp no)
-		(fields_autoplaced yes)
-		(property "Reference" "U2"
-			(at 133.35 69.85 0)
-			(effects
-				(font
-					(size 1.27 1.27)
-				)
-			)
-		)
-		(property "Value" "6N138"
-			(at 133.35 72.39 0)
-			(effects
-				(font
-					(size 1.27 1.27)
-				)
-			)
-		)
-		(property "Footprint" ""
-			(at 140.716 90.17 0)
-			(effects
-				(font
-					(size 1.27 1.27)
-				)
-				(hide yes)
-			)
-		)
-		(property "Datasheet" "http://www.onsemi.com/pub/Collateral/HCPL2731-D.pdf"
-			(at 140.716 90.17 0)
-			(effects
-				(font
-					(size 1.27 1.27)
-				)
-				(hide yes)
-			)
-		)
-		(property "Description" "Low Input Current high Gain Split Darlington Optocouplers, -0.5V to 7V VDD, DIP-8"
-			(at 133.35 82.55 0)
-			(effects
-				(font
-					(size 1.27 1.27)
-				)
-				(hide yes)
-			)
-		)
-		(pin "6"
-		)
-		(pin "8"
-		)
-		(pin "5"
-		)
-		(pin "2"
-		)
-		(pin "7"
-		)
-		(pin "3"
-		)
-		(pin "4"
-		)
-		(pin "1"
-		)
-		(instances
-			(project ""
-				(path "/11b6b3e0-6260-4ffa-b9c7-47f3b03473c9/e71ecf15-c300-4c9d-862f-92665ebf3933/d2fa69c2-c3e0-43db-84db-bb1b3a6e2002"
-					(reference "U2")
-					(unit 1)
-				)
-			)
-		)
-	)
-	(symbol
 		(lib_id "Diode:1N4001")
 		(at 111.76 85.09 270)
@@
 	(symbol
 		(lib_id "power:GND")
-		(at 140.97 90.17 0)
+		(at 133.35 95.25 0)
 		(unit 1)
 		(exclude_from_sim no)
@@
 		(fields_autoplaced yes)
 		(property "Reference" "#PWR05"
-			(at 140.97 96.52 0)
+			(at 133.35 101.6 0)
 			(effects
 				(font
@@
 		)
 		(property "Value" "GND"
-			(at 140.97 95.25 0)
+			(at 133.35 100.33 0)
 			(effects
 				(font
@@
 		)
 		(property "Footprint" ""
-			(at 140.97 90.17 0)
+			(at 133.35 95.25 0)
 			(effects
 				(font
@@
 		)
 		(property "Datasheet" ""
-			(at 140.97 90.17 0)
+			(at 133.35 95.25 0)
 			(effects
 				(font
@@
 		)
 		(property "Description" "Power symbol creates a global label with name \"GND\" , ground"
-			(at 140.97 90.17 0)
-			(effects
-				(font
+			(at 133.35 95.25 0)
+			(effects
+				(font
