File: kicad/led.kicad_sch (KiCad schematic)
At the start: 3 parts

Commit message: kicad changes
Parts:
- renumbered C4 to C8, R10 to R17
Changed lines of the file:
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@@
 		(dnp no)
 		(fields_autoplaced yes)
-		(property "Reference" "R10"
+		(property "Reference" "R17"
 			(at 109.22 39.37 90)
 			(effects
@@
 		)
 		(instances
-			(project ""
-				(path "/11b6b3e0-6260-4ffa-b9c7-47f3b03473c9/e71ecf15-c300-4c9d-862f-92665ebf3933/bce221a1-3f98-4830-92f6-4b4f6a4941ad"
-					(reference "R10")
+			(project "dcc"
+				(path "/11b6b3e0-6260-4ffa-b9c7-47f3b03473c9/e71ecf15-c300-4c9d-862f-92665ebf3933/3c3350b0-7269-44ea-ac7b-f964376fa21d"
+					(reference "R18")
+					(unit 1)
+				)
+				(path "/11b6b3e0-6260-4ffa-b9c7-47f3b03473c9/e71ecf15-c300-4c9d-862f-92665ebf3933/4719d1eb-cf2d-47ff-b071-3767ef61e3e8"
+					(reference "R17")
 					(unit 1)
 				)
@@
 		(dnp no)
 		(fields_autoplaced yes)
-		(property "Reference" "C4"
+		(property "Reference" "C8"
 			(at 118.11 57.15 0)
 			(effects
@@
 		)
 		(instances
-			(project ""
-				(path "/11b6b3e0-6260-4ffa-b9c7-47f3b03473c9/e71ecf15-c300-4c9d-862f-92665ebf3933/bce221a1-3f98-4830-92f6-4b4f6a4941ad"
-					(reference "C4")
+			(project "dcc"
+				(path "/11b6b3e0-6260-4ffa-b9c7-47f3b03473c9/e71ecf15-c300-4c9d-862f-92665ebf3933/3c3350b0-7269-44ea-ac7b-f964376fa21d"
+					(reference "C9")
+					(unit 1)
+				)
+				(path "/11b6b3e0-6260-4ffa-b9c7-47f3b03473c9/e71ecf15-c300-4c9d-862f-92665ebf3933/4719d1eb-cf2d-47ff-b071-3767ef61e3e8"
+					(reference "C8")
 					(unit 1)
 				)
@@
 		(dnp no)
 		(fields_autoplaced yes)
-		(property "Reference" "#PWR09"
+		(property "Reference" "#PWR014"
 			(at 105.41 96.52 0)
 			(effects
@@
 		)
 		(instances
-			(project ""
-				(path "/11b6b3e0-6260-4ffa-b9c7-47f3b03473c9/e71ecf15-c300-4c9d-862f-92665ebf3933/bce221a1-3f98-4830-92f6-4b4f6a4941ad"
-					(reference "#PWR09")
+			(project "dcc"
+				(path "/11b6b3e0-6260-4ffa-b9c7-47f3b03473c9/e71ecf15-c300-4c9d-862f-92665ebf3933/3c3350b0-7269-44ea-ac7b-f964376fa21d"
+					(reference "#PWR018")
+					(unit 1)
+				)
+				(path "/11b6b3e0-6260-4ffa-b9c7-47f3b03473c9/e71ecf15-c300-4c9d-862f-92665ebf3933/4719d1eb-cf2d-47ff-b071-3767ef61e3e8"
+					(reference "#PWR014")
 					(unit 1)
 				)
@@
 		(instances
 			(project "dcc"
+				(path "/11b6b3e0-6260-4ffa-b9c7-47f3b03473c9/e71ecf15-c300-4c9d-862f-92665ebf3933/3c3350b0-7269-44ea-ac7b-f964376fa21d"
+					(reference "#PWR019")
+					(unit 1)
+				)
+				(path "/11b6b3e0-6260-4ffa-b9c7-47f3b03473c9/e71ecf15-c300-4c9d-862f-92665ebf3933/4719d1eb-cf2d-47ff-b071-3767ef61e3e8"
+					(reference "#PWR017")
+					(unit 1)
+				)
 				(path "/11b6b3e0-6260-4ffa-b9c7-47f3b03473c9/e71ecf15-c300-4c9d-862f-92665ebf3933/bce221a1-3f98-4830-92f6-4b4f6a4941ad"
 					(reference "#PWR010")
@@
 		(instances
 			(project "dcc"
+				(path "/11b6b3e0-6260-4ffa-b9c7-47f3b03473c9/e71ecf15-c300-4c9d-862f-92665ebf3933/3c3350b0-7269-44ea-ac7b-f964376fa21d"
+					(reference "D6")
+					(unit 1)
+				)
+				(path "/11b6b3e0-6260-4ffa-b9c7-47f3b03473c9/e71ecf15-c300-4c9d-862f-92665ebf3933/4719d1eb-cf2d-47ff-b071-3767ef61e3e8"
+					(reference "D4")
+					(unit 1)
+				)
 				(path "/11b6b3e0-6260-4ffa-b9c7-47f3b03473c9/e71ecf15-c300-4c9d-862f-92665ebf3933/bce221a1-3f98-4830-92f6-4b4f6a4941ad"
 					(reference "D10")
