File: kicad/power.kicad_sch (KiCad schematic)
At the start: 0 parts

Commit message: split
Parts:
- added C2: 470uF, symbol Device:C_Polarized_US
- added C3: 0.1uF, symbol Device:C_Polarized_US
- added D1: MB6S, Package_TO_SOT_SMD:TO-269AA, symbol Diode_Bridge:MB6S
- added D3, D4: 1N4001, Diode_THT:D_DO-41_SOD81_P10.16mm_Horizontal, symbol Diode:1N4001
- added R8: 10K, symbol Device:R
- added U1: LD1117S50TR_SOT223, Package_TO_SOT_SMD:SOT-223-3_TabPin2, symbol Regulator_Linear:LD1117S50TR_SOT223
Connections:
- new net: C3.1, D3.2 (A), U1.2 (VO)
- new net: C2.1, D1.3 (+), D4.2 (A), R8.1, U1.3 (VI)
- new net 12V: D4.1 (K)
- new net 5V: D3.1 (K)
- new net GND: C2.2, C3.2, D1.4 (-), R8.2, U1.1 (GND)
- new net RAIL_1: D1.2
- new net RAIL_2: D1.1
Other:
- note added: "800mA"
- note added: "https://electronics.stackexchange.com/a/14408"
- note added: "https://www.engineersedge.com/instrumentation/capacitance_discharge/capacitance_discharge_calculator_12909.htm"

Commit message: kicad changes
Parts:
- removed D3, D4: 1N4001, Diode_THT:D_DO-41_SOD81_P10.16mm_Horizontal, symbol Diode:1N4001
- C2: value 470uF -> 47uF
Connections:
- net 12V: now also C2.1, D1.3 (+), R8.1, U1.3 (VI)
- net 5V: now also C3.1, U1.2 (VO)
Other:
- note added: "Actual ~9-10V"
Changed lines of the file:
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@@
-	(wire
-		(pts
-			(xy 203.2 34.29) (xy 203.2 43.18)
-		)
-		(stroke
-			(width 0)
-			(type default)
-		)
-	)
 	(wire
 		(pts
@@
 	(wire
 		(pts
-			(xy 203.2 50.8) (xy 203.2 76.2)
+			(xy 203.2 34.29) (xy 203.2 76.2)
 		)
 		(stroke
@@
 	(wire
 		(pts
-			(xy 168.91 49.53) (xy 168.91 76.2)
+			(xy 168.91 33.02) (xy 168.91 76.2)
 		)
 		(stroke
@@
 	(wire
 		(pts
-			(xy 168.91 33.02) (xy 168.91 41.91)
-		)
-		(stroke
-			(width 0)
-			(type default)
-		)
-	)
-	(wire
-		(pts
 			(xy 168.91 86.36) (xy 168.91 90.17)
 		)
@@
 			(width 0)
 			(type default)
+		)
+	)
+	(text "Actual ~9-10V\n"
+		(exclude_from_sim no)
+		(at 161.036 32.258 0)
+		(effects
+			(font
+				(size 1.27 1.27)
+			)
 		)
 	)
@@
 			)
 			(justify right)
-		)
-	)
-	(symbol
-		(lib_id "Diode:1N4001")
-		(at 203.2 46.99 270)
-		(unit 1)
-		(exclude_from_sim no)
-		(in_bom yes)
-		(on_board yes)
-		(dnp no)
-		(fields_autoplaced yes)
-		(property "Reference" "D3"
-			(at 205.74 45.72 90)
-			(effects
-				(font
-					(size 1.27 1.27)
-				)
-				(justify left)
-			)
-		)
-		(property "Value" "1N4001"
-			(at 205.74 48.26 90)
-			(effects
-				(font
-					(size 1.27 1.27)
-				)
-				(justify left)
-			)
-		)
-		(property "Footprint" "Diode_THT:D_DO-41_SOD81_P10.16mm_Horizontal"
-			(at 203.2 46.99 0)
-			(effects
-				(font
-					(size 1.27 1.27)
-				)
-				(hide yes)
-			)
-		)
-		(property "Datasheet" "http://www.vishay.com/docs/88503/1n4001.pdf"
-			(at 203.2 46.99 0)
-			(effects
-				(font
-					(size 1.27 1.27)
-				)
-				(hide yes)
-			)
-		)
-		(property "Description" "50V 1A General Purpose Rectifier Diode, DO-41"
-			(at 203.2 46.99 0)
-			(effects
-				(font
-					(size 1.27 1.27)
-				)
-				(hide yes)
-			)
-		)
-		(property "Sim.Device" "D"
-			(at 203.2 46.99 0)
-			(effects
-				(font
-					(size 1.27 1.27)
-				)
-				(hide yes)
-			)
-		)
-		(property "Sim.Pins" "1=K 2=A"
-			(at 203.2 46.99 0)
-			(effects
-				(font
-					(size 1.27 1.27)
-				)
-				(hide yes)
-			)
-		)
-		(pin "1"
-		)
-		(pin "2"
-		)
-		(instances
-			(project ""
-				(path "/11b6b3e0-6260-4ffa-b9c7-47f3b03473c9/e71ecf15-c300-4c9d-862f-92665ebf3933/fe0267e8-6263-40e8-a151-ccbc1a5c7034"
-					(reference "D3")
-					(unit 1)
-				)
-			)
 		)
 	)
@@
 	)
 	(symbol
-		(lib_id "Diode:1N4001")
-		(at 168.91 45.72 270)
-		(unit 1)
-		(exclude_from_sim no)
-		(in_bom yes)
-		(on_board yes)
-		(dnp no)
-		(fields_autoplaced yes)
-		(property "Reference" "D4"
-			(at 171.45 44.45 90)
-			(effects
-				(font
-					(size 1.27 1.27)
-				)
-				(justify left)
-			)
-		)
-		(property "Value" "1N4001"
-			(at 171.45 46.99 90)
-			(effects
-				(font
-					(size 1.27 1.27)
-				)
-				(justify left)
-			)
-		)
-		(property "Footprint" "Diode_THT:D_DO-41_SOD81_P10.16mm_Horizontal"
-			(at 168.91 45.72 0)
-			(effects
-				(font
-					(size 1.27 1.27)
-				)
-				(hide yes)
-			)
-		)
-		(property "Datasheet" "http://www.vishay.com/docs/88503/1n4001.pdf"
-			(at 168.91 45.72 0)
-			(effects
-				(font
-					(size 1.27 1.27)
-				)
-				(hide yes)
-			)
-		)
-		(property "Description" "50V 1A General Purpose Rectifier Diode, DO-41"
-			(at 168.91 45.72 0)
-			(effects
-				(font
-					(size 1.27 1.27)
-				)
-				(hide yes)
-			)
-		)
-		(property "Sim.Device" "D"
-			(at 168.91 45.72 0)
-			(effects
-				(font
-					(size 1.27 1.27)
-				)
-				(hide yes)
-			)
-		)
-		(property "Sim.Pins" "1=K 2=A"
-			(at 168.91 45.72 0)
-			(effects
-				(font
-					(size 1.27 1.27)
-				)
-				(hide yes)
-			)
-		)
-		(pin "1"
-		)
-		(pin "2"
-		)
-		(instances
-			(project "dcc"
-				(path "/11b6b3e0-6260-4ffa-b9c7-47f3b03473c9/e71ecf15-c300-4c9d-862f-92665ebf3933/fe0267e8-6263-40e8-a151-ccbc1a5c7034"
-					(reference "D4")
-					(unit 1)
-				)
-			)
-		)
-	)
-	(symbol
 		(lib_id "power:GND")
 		(at 184.15 92.71 0)
@@
 			)
 		)
-		(property "Value" "470uF"
+		(property "Value" "47uF"
 			(at 158.75 83.185 0)
 			(effects
