File: kicad/transmitter.kicad_sch (KiCad schematic)
At the start: 1 part, among them SW1 SW

Commit message: new screen, minimum functional
Other:
- sheet Inverter renamed Inverter A
- sheet Inverter1 renamed Inverter B
- sheet Motor controller renamed Motor controller (L298N)
- removed sheet Screen
- added sheet Screen (SSD1322) (screen_ssd1322.kicad_sch)

Commit message: kicad changes
Parts:
- added SW3: SW, symbol Switch:SW_DPDT_x2
Connections:
- net +12V: now also SW3.2 (B)
- new net Motor controller (L298N)1/VCC_12V: SW3.1 (A)
- no-connect marks 1 -> 2
Other:
- added sheet Button (button.kicad_sch)
- added sheet Button1 (button.kicad_sch)
- added sheet Button2 (button.kicad_sch)
- added sheet ESP32-C6 (esp32-c6.kicad_sch)
- added sheet Inverter A1 (inverter.kicad_sch)
- added sheet Inverter A2 (inverter.kicad_sch)
- added sheet Motor controller (L298N)1 (motor_controller.kicad_sch)
- added sheet Rotary encoder1 (rotary_encoder.kicad_sch)
- added sheet Screen (SSD1322)1 (screen_ssd1322.kicad_sch)
