File: kicad/button.kicad_sch (KiCad schematic)
At the start: 3 parts, among them Q2 2N3904

Commit message: kicad changes
Parts:
- removed Q2: 2N3904, Package_TO_SOT_THT:TO-92_Inline, symbol Transistor_BJT:2N3904
- removed R3, R4: 1k, symbol Device:R
- added C6: 100nF, symbol Device:C
- added R14: 10K, symbol Device:R
- added SW4: SW_Push, symbol Switch:SW_Push
Connections:
- net GND: now also C6.2, R14.1
- new net OUT: C6.1, R14.2, SW4.2
- new net VCC: SW4.1
Other:
- note removed: "https://dcc-ex.com/reference/hardware/motorboards/L298N-motor-board-setup.html"

Commit message: c6 buttons rework
Parts:
- C6: value 100nF -> 0.1uF
Changed lines of the file:
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@@
 			)
 		)
-		(property "Value" "100nF"
+		(property "Value" "0.1uF"
 			(at 118.11 97.79 0)
 			(effects
