File: kicad/esp32-c6.kicad_sch (KiCad schematic)
At the start: 0 parts

Commit message: c6 buttons rework
Other:
- note added: "8 is LED"
- note removed: "Pin 14? LED?"
Changed lines of the file:
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@@
 	(generator_version "8.0")
 	(paper "A4")
-	(text "Pin 14? LED?\n"
+	(text "8 is LED"
 		(exclude_from_sim no)
-		(at 91.186 130.81 0)
+		(at 100.584 116.078 0)
 		(effects
 			(font
